Commit message: Royal Park trees from the point cloud: textured crown shells rounded underneath, trunks under crown tops, shrubs to the ground; sky
Co-Authored-By: Claude Opus 5.5 (1M context) <noreply@anthropic.com>

File: scout_navigation/worlds/royal_park.sdf.xacro (robot description, xacro)
@@ -17,5 +17,5 @@
         <ambient_light>0.4 0.4 0.4</ambient_light>
         <background_color>0.7 0.8 0.9</background_color>
-        <camera_pose>-12 -10 8 0 0.45 0.6</camera_pose>
+        <camera_pose>25 -32 24 0 0.55 1.5708</camera_pose>
       </plugin>
       <plugin filename="GzSceneManager" name="Scene Manager">
@@ -120,4 +120,8 @@
             name="ignition::gazebo::systems::NavSat"/>
     <!-- Grid origin sits on the survey start point used by survey_navigator -->
+    <scene>
+      <ambient>0.6 0.6 0.6 1</ambient>
+      <sky></sky>
+    </scene>
     <spherical_coordinates>
       <surface_model>EARTH_WGS84</surface_model>
@@ -144,147 +148,65 @@
         </visual>
       </link>
-      <link name="tree_0">
-        <pose>-22.09 -15.10 -1.34 0 0 0</pose>
-        <collision name="trunk"><pose>0 0 0.25 0 0 0</pose>
-          <geometry><cylinder><radius>0.2</radius><length>4.5</length></cylinder></geometry>
+      <link name="vegetation">
+        <collision name="collision">
+          <geometry><mesh><uri>file://$(arg share)/worlds/royal_park/objects.obj</uri></mesh></geometry>
         </collision>
-        <visual name="trunk"><pose>0 0 0.25 0 0 0</pose>
-          <geometry><cylinder><radius>0.2</radius><length>4.5</length></cylinder></geometry>
-          <material><ambient>0.35 0.25 0.15 1</ambient><diffuse>0.35 0.25 0.15 1</diffuse></material></visual>
-        <visual name="crown"><pose>0 0 7.88 0 0 0</pose>
-          <geometry><sphere><radius>1.60</radius></sphere></geometry>
-          <material><ambient>0.2 0.35 0.15 0.6</ambient><diffuse>0.2 0.35 0.15 0.6</diffuse></material></visual>
-      </link>
-      <link name="tree_1">
-        <pose>-10.07 -14.36 -1.08 0 0 0</pose>
-        <collision name="trunk"><pose>0 0 0.25 0 0 0</pose>
-          <geometry><cylinder><radius>0.2</radius><length>4.5</length></cylinder></geometry>
-        </collision>
-        <visual name="trunk"><pose>0 0 0.25 0 0 0</pose>
-          <geometry><cylinder><radius>0.2</radius><length>4.5</length></cylinder></geometry>
-          <material><ambient>0.35 0.25 0.15 1</ambient><diffuse>0.35 0.25 0.15 1</diffuse></material></visual>
-        <visual name="crown"><pose>0 0 5.18 0 0 0</pose>
-          <geometry><sphere><radius>1.95</radius></sphere></geometry>
-          <material><ambient>0.2 0.35 0.15 0.6</ambient><diffuse>0.2 0.35 0.15 0.6</diffuse></material></visual>
-      </link>
-      <link name="tree_2">
-        <pose>-25.45 -9.02 -1.27 0 0 0</pose>
-        <collision name="trunk"><pose>0 0 0.25 0 0 0</pose>
-          <geometry><cylinder><radius>0.2</radius><length>4.5</length></cylinder></geometry>
-        </collision>
-        <visual name="trunk"><pose>0 0 0.25 0 0 0</pose>
-          <geometry><cylinder><radius>0.2</radius><length>4.5</length></cylinder></geometry>
-          <material><ambient>0.35 0.25 0.15 1</ambient><diffuse>0.35 0.25 0.15 1</diffuse></material></visual>
-        <visual name="crown"><pose>0 0 10.09 0 0 0</pose>
-          <geometry><sphere><radius>3.83</radius></sphere></geometry>
-          <material><ambient>0.2 0.35 0.15 0.6</ambient><diffuse>0.2 0.35 0.15 0.6</diffuse></material></visual>
-      </link>
-      <link name="tree_3">
-        <pose>-28.90 -6.45 -1.20 0 0 0</pose>
-        <collision name="trunk"><pose>0 0 0.25 0 0 0</pose>
-          <geometry><cylinder><radius>0.2</radius><length>4.5</length></cylinder></geometry>
-        </collision>
-        <visual name="trunk"><pose>0 0 0.25 0 0 0</pose>
-          <geometry><cylinder><radius>0.2</radius><length>4.5</length></cylinder></geometry>
-          <material><ambient>0.35 0.25 0.15 1</ambient><diffuse>0.35 0.25 0.15 1</diffuse></material></visual>
-        <visual name="crown"><pose>0 0 10.59 0 0 0</pose>
-          <geometry><sphere><radius>3.83</radius></sphere></geometry>
-          <material><ambient>0.2 0.35 0.15 0.6</ambient><diffuse>0.2 0.35 0.15 0.6</diffuse></material></visual>
-      </link>
-      <link name="tree_4">
-        <pose>-5.84 -3.95 -0.19 0 0 0</pose>
-        <collision name="trunk"><pose>0 0 0.25 0 0 0</pose>
-          <geometry><cylinder><radius>0.2</radius><length>4.5</length></cylinder></geometry>
-        </collision>
-        <visual name="trunk"><pose>0 0 0.25 0 0 0</pose>
-          <geometry><cylinder><radius>0.2</radius><length>4.5</length></cylinder></geometry>
-          <material><ambient>0.35 0.25 0.15 1</ambient><diffuse>0.35 0.25 0.15 1</diffuse></material></visual>
-        <visual name="crown"><pose>0 0 8.17 0 0 0</pose>
-          <geometry><sphere><radius>3.74</radius></sphere></geometry>
-          <material><ambient>0.2 0.35 0.15 0.6</ambient><diffuse>0.2 0.35 0.15 0.6</diffuse></material></visual>
-      </link>
-      <link name="tree_5">
-        <pose>23.91 52.41 0.99 0 0 0</pose>
-        <collision name="trunk"><pose>0 0 0.25 0 0 0</pose>
-          <geometry><cylinder><radius>0.2</radius><length>4.5</length></cylinder></geometry>
-        </collision>
-        <visual name="trunk"><pose>0 0 0.25 0 0 0</pose>
-          <geometry><cylinder><radius>0.2</radius><length>4.5</length></cylinder></geometry>
-          <material><ambient>0.35 0.25 0.15 1</ambient><diffuse>0.35 0.25 0.15 1</diffuse></material></visual>
-        <visual name="crown"><pose>0 0 11.58 0 0 0</pose>
-          <geometry><sphere><radius>3.52</radius></sphere></geometry>
-          <material><ambient>0.2 0.35 0.15 0.6</ambient><diffuse>0.2 0.35 0.15 0.6</diffuse></material></visual>
-      </link>
-      <link name="tree_6">
-        <pose>0.66 64.42 1.04 0 0 0</pose>
-        <collision name="trunk"><pose>0 0 0.25 0 0 0</pose>
-          <geometry><cylinder><radius>0.2</radius><length>4.5</length></cylinder></geometry>
-        </collision>
-        <visual name="trunk"><pose>0 0 0.25 0 0 0</pose>
-          <geometry><cylinder><radius>0.2</radius><length>4.5</length></cylinder></geometry>
-          <material><ambient>0.35 0.25 0.15 1</ambient><diffuse>0.35 0.25 0.15 1</diffuse></material></visual>
-        <visual name="crown"><pose>0 0 1.76 0 0 0</pose>
-          <geometry><sphere><radius>0.80</radius></sphere></geometry>
-          <material><ambient>0.2 0.35 0.15 0.6</ambient><diffuse>0.2 0.35 0.15 0.6</diffuse></material></visual>
-      </link>
-      <link name="tree_7">
-        <pose>-11.32 65.19 0.84 0 0 0</pose>
-        <collision name="trunk"><pose>0 0 0.25 0 0 0</pose>
-          <geometry><cylinder><radius>0.2</radius><length>4.5</length></cylinder></geometry>
-        </collision>
-        <visual name="trunk"><pose>0 0 0.25 0 0 0</pose>
-          <geometry><cylinder><radius>0.2</radius><length>4.5</length></cylinder></geometry>
-          <material><ambient>0.35 0.25 0.15 1</ambient><diffuse>0.35 0.25 0.15 1</diffuse></material></visual>
-        <visual name="crown"><pose>0 0 7.08 0 0 0</pose>
-          <geometry><sphere><radius>0.49</radius></sphere></geometry>
-          <material><ambient>0.2 0.35 0.15 0.6</ambient><diffuse>0.2 0.35 0.15 0.6</diffuse></material></visual>
-      </link>
-      <link name="tree_8">
-        <pose>-6.82 65.09 0.86 0 0 0</pose>
-        <collision name="trunk"><pose>0 0 0.25 0 0 0</pose>
-          <geometry><cylinder><radius>0.2</radius><length>4.5</length></cylinder></geometry>
-        </collision>
-        <visual name="trunk"><pose>0 0 0.25 0 0 0</pose>
-          <geometry><cylinder><radius>0.2</radius><length>4.5</length></cylinder></geometry>
-          <material><ambient>0.35 0.25 0.15 1</ambient><diffuse>0.35 0.25 0.15 1</diffuse></material></visual>
-        <visual name="crown"><pose>0 0 6.78 0 0 0</pose>
-          <geometry><sphere><radius>1.62</radius></sphere></geometry>
-          <material><ambient>0.2 0.35 0.15 0.6</ambient><diffuse>0.2 0.35 0.15 0.6</diffuse></material></visual>
-      </link>
-      <link name="tree_9">
-        <pose>-6.32 65.08 0.86 0 0 0</pose>
-        <collision name="trunk"><pose>0 0 0.25 0 0 0</pose>
-          <geometry><cylinder><radius>0.2</radius><length>4.5</length></cylinder></geometry>
-        </collision>
-        <visual name="trunk"><pose>0 0 0.25 0 0 0</pose>
-          <geometry><cylinder><radius>0.2</radius><length>4.5</length></cylinder></geometry>
-          <material><ambient>0.35 0.25 0.15 1</ambient><diffuse>0.35 0.25 0.15 1</diffuse></material></visual>
-        <visual name="crown"><pose>0 0 6.78 0 0 0</pose>
-          <geometry><sphere><radius>1.62</radius></sphere></geometry>
-          <material><ambient>0.2 0.35 0.15 0.6</ambient><diffuse>0.2 0.35 0.15 0.6</diffuse></material></visual>
-      </link>
-      <link name="tree_10">
-        <pose>25.67 64.37 1.02 0 0 0</pose>
-        <collision name="trunk"><pose>0 0 0.25 0 0 0</pose>
-          <geometry><cylinder><radius>0.2</radius><length>4.5</length></cylinder></geometry>
-        </collision>
-        <visual name="trunk"><pose>0 0 0.25 0 0 0</pose>
-          <geometry><cylinder><radius>0.2</radius><length>4.5</length></cylinder></geometry>
-          <material><ambient>0.35 0.25 0.15 1</ambient><diffuse>0.35 0.25 0.15 1</diffuse></material></visual>
-        <visual name="crown"><pose>0 0 4.74 0 0 0</pose>
-          <geometry><sphere><radius>2.84</radius></sphere></geometry>
-          <material><ambient>0.2 0.35 0.15 0.6</ambient><diffuse>0.2 0.35 0.15 0.6</diffuse></material></visual>
-      </link>
-      <link name="tree_11">
-        <pose>29.67 64.28 1.04 0 0 0</pose>
-        <collision name="trunk"><pose>0 0 0.25 0 0 0</pose>
-          <geometry><cylinder><radius>0.2</radius><length>4.5</length></cylinder></geometry>
-        </collision>
-        <visual name="trunk"><pose>0 0 0.25 0 0 0</pose>
-          <geometry><cylinder><radius>0.2</radius><length>4.5</length></cylinder></geometry>
-          <material><ambient>0.35 0.25 0.15 1</ambient><diffuse>0.35 0.25 0.15 1</diffuse></material></visual>
-        <visual name="crown"><pose>0 0 4.77 0 0 0</pose>
-          <geometry><sphere><radius>2.84</radius></sphere></geometry>
-          <material><ambient>0.2 0.35 0.15 0.6</ambient><diffuse>0.2 0.35 0.15 0.6</diffuse></material></visual>
+        <visual name="visual">
+          <geometry><mesh><uri>file://$(arg share)/worlds/royal_park/objects.obj</uri></mesh></geometry>
+        </visual>
+      </link>
+      <link name="trunk_0">
+        <pose>-22.70 -14.71 2.20 0 0 0</pose>
+        <collision name="collision"><geometry><cylinder><radius>0.11</radius><length>7.46</length></cylinder></geometry></collision>
+        <visual name="visual"><geometry><cylinder><radius>0.11</radius><length>7.46</length></cylinder></geometry>
+          <material><ambient>0.30 0.22 0.15 1</ambient><diffuse>0.36 0.27 0.18 1</diffuse></material></visual>
+      </link>
+      <link name="trunk_1">
+        <pose>-9.93 -13.99 1.07 0 0 0</pose>
+        <collision name="collision"><geometry><cylinder><radius>0.14</radius><length>4.63</length></cylinder></geometry></collision>
+        <visual name="visual"><geometry><cylinder><radius>0.14</radius><length>4.63</length></cylinder></geometry>
+          <material><ambient>0.30 0.22 0.15 1</ambient><diffuse>0.36 0.27 0.18 1</diffuse></material></visual>
+      </link>
+      <link name="trunk_2">
+        <pose>-25.58 -8.89 3.35 0 0 0</pose>
+        <collision name="collision"><geometry><cylinder><radius>0.21</radius><length>9.71</length></cylinder></geometry></collision>
+        <visual name="visual"><geometry><cylinder><radius>0.21</radius><length>9.71</length></cylinder></geometry>
+          <material><ambient>0.30 0.22 0.15 1</ambient><diffuse>0.36 0.27 0.18 1</diffuse></material></visual>
+      </link>
+      <link name="trunk_3">
+        <pose>-29.28 -6.81 3.49 0 0 0</pose>
+        <collision name="collision"><geometry><cylinder><radius>0.21</radius><length>9.94</length></cylinder></geometry></collision>
+        <visual name="visual"><geometry><cylinder><radius>0.21</radius><length>9.94</length></cylinder></geometry>
+          <material><ambient>0.30 0.22 0.15 1</ambient><diffuse>0.36 0.27 0.18 1</diffuse></material></visual>
+      </link>
+      <link name="trunk_4">
+        <pose>-5.94 -3.07 3.19 0 0 0</pose>
+        <collision name="collision"><geometry><cylinder><radius>0.32</radius><length>7.06</length></cylinder></geometry></collision>
+        <visual name="visual"><geometry><cylinder><radius>0.32</radius><length>7.06</length></cylinder></geometry>
+          <material><ambient>0.30 0.22 0.15 1</ambient><diffuse>0.36 0.27 0.18 1</diffuse></material></visual>
+      </link>
+      <link name="trunk_5">
+        <pose>23.78 52.54 5.48 0 0 0</pose>
+        <collision name="collision"><geometry><cylinder><radius>0.29</radius><length>9.41</length></cylinder></geometry></collision>
+        <visual name="visual"><geometry><cylinder><radius>0.29</radius><length>9.41</length></cylinder></geometry>
+          <material><ambient>0.30 0.22 0.15 1</ambient><diffuse>0.36 0.27 0.18 1</diffuse></material></visual>
+      </link>
+      <link name="trunk_6">
+        <pose>18.93 59.39 4.07 0 0 0</pose>
+        <collision name="collision"><geometry><cylinder><radius>0.21</radius><length>6.67</length></cylinder></geometry></collision>
+        <visual name="visual"><geometry><cylinder><radius>0.21</radius><length>6.67</length></cylinder></geometry>
+          <material><ambient>0.30 0.22 0.15 1</ambient><diffuse>0.36 0.27 0.18 1</diffuse></material></visual>
+      </link>
+      <link name="trunk_7">
+        <pose>25.79 64.00 2.98 0 0 0</pose>
+        <collision name="collision"><geometry><cylinder><radius>0.21</radius><length>4.41</length></cylinder></geometry></collision>
+        <visual name="visual"><geometry><cylinder><radius>0.21</radius><length>4.41</length></cylinder></geometry>
+          <material><ambient>0.30 0.22 0.15 1</ambient><diffuse>0.36 0.27 0.18 1</diffuse></material></visual>
+      </link>
+      <link name="trunk_8">
+        <pose>-6.71 64.46 4.68 0 0 0</pose>
+        <collision name="collision"><geometry><cylinder><radius>0.10</radius><length>8.15</length></cylinder></geometry></collision>
+        <visual name="visual"><geometry><cylinder><radius>0.10</radius><length>8.15</length></cylinder></geometry>
+          <material><ambient>0.30 0.22 0.15 1</ambient><diffuse>0.36 0.27 0.18 1</diffuse></material></visual>
       </link>
     </model>
