Commit message: Driven U-turns for the towed train: midpoint-pivot hitch geometry, turn design study, headland runs, no stop between line and turn; Rx ground clearance and cart wheel friction fixed
Co-Authored-By: Claude Opus 5.5 (1M context) <noreply@anthropic.com>

File: scout_navigation/description/temrover_carts.xacro (robot description, xacro)
@@ -9,5 +9,5 @@
     <xacro:property name="yaw_limit" value="1.2" />
     <xacro:property name="pitch_limit" value="0.5" />
-    <xacro:macro name="cart_wheel" params="cart name *origin">
+    <xacro:macro name="cart_wheel" params="cart name *origin lateral_friction:=0.6">
         <link name="${cart}_${name}_wheel_link">
             <inertial>
@@ -35,30 +35,52 @@
         </joint>
         <gazebo reference="${cart}_${name}_wheel_link">
+            <!-- fdir1 in the wheel frame, so mu1 acts along the rolling direction -->
+            <fdir1>1 0 0</fdir1>
             <mu1>0.8</mu1>
-            <mu2>0.6</mu2>
+            <mu2>${lateral_friction}</mu2>
             <material>Gazebo/DarkGrey</material>
         </gazebo>
     </xacro:macro>
-    <!-- Yaw then pitch, matching the four hitch degrees of freedom of the Simscape model -->
+    <!-- Each PVC link is two rigid V frames pinned at its midpoint: the front half is fixed to the
+         towing unit, the yaw joint sits halfway, and the rear half pitches with the towed cart -->
     <xacro:macro name="cart_body" params="cart parent mass length width height
                                           tow_x tow_z rod front_x front_z">
+        <link name="${cart}_tow_link">
+            <inertial>
+                <origin xyz="${-rod/4} 0 0" />
+                <mass value="2.0" />
+                <inertia ixx="0.01" ixy="0" ixz="0" iyy="${2.0*rod*rod/48}" iyz="0"
+                         izz="${2.0*rod*rod/48}" />
+            </inertial>
+            <visual>
+                <origin xyz="${-rod/4} 0 0" rpy="0 ${pi/2} 0" />
+                <geometry>
+                    <cylinder length="${rod/2}" radius="0.02" />
+                </geometry>
+            </visual>
+        </link>
+        <joint name="${cart}_tow_frame" type="fixed">
+            <parent link="${parent}" />
+            <child link="${cart}_tow_link" />
+            <origin xyz="${tow_x} 0 ${tow_z}" />
+        </joint>
         <link name="${cart}_rod_link">
             <inertial>
-                <origin xyz="${-rod/2} 0 0" />
-                <mass value="4.0" />
-                <inertia ixx="0.01" ixy="0" ixz="0" iyy="${4.0*rod*rod/12}" iyz="0"
-                         izz="${4.0*rod*rod/12}" />
+                <origin xyz="${-rod/4} 0 0" />
+                <mass value="2.0" />
+                <inertia ixx="0.01" ixy="0" ixz="0" iyy="${2.0*rod*rod/48}" iyz="0"
+                         izz="${2.0*rod*rod/48}" />
             </inertial>
             <visual>
-                <origin xyz="${-rod/2} 0 0" rpy="0 ${pi/2} 0" />
+                <origin xyz="${-rod/4} 0 0" rpy="0 ${pi/2} 0" />
                 <geometry>
-                    <cylinder length="${rod}" radius="0.02" />
+                    <cylinder length="${rod/2}" radius="0.02" />
                 </geometry>
             </visual>
         </link>
         <joint name="${cart}_hitch_yaw" type="revolute">
-            <parent link="${parent}" />
+            <parent link="${cart}_tow_link" />
             <child link="${cart}_rod_link" />
-            <origin xyz="${tow_x} 0 ${tow_z}" />
+            <origin xyz="${-rod/2} 0 0" />
             <axis xyz="0 0 1" />
             <limit lower="${-yaw_limit}" upper="${yaw_limit}" effort="500" velocity="10" />
@@ -94,5 +116,5 @@
             <parent link="${cart}_rod_link" />
             <child link="${cart}_link" />
-            <origin xyz="${-rod-front_x} 0 ${front_z}" />
+            <origin xyz="${-rod/2-front_x} 0 ${front_z}" />
             <axis xyz="0 1 0" />
             <limit lower="${-pitch_limit}" upper="${pitch_limit}" effort="500" velocity="10" />
@@ -116,7 +138,8 @@
         <origin xyz="-0.700 -0.300 -0.215" />
     </xacro:cart_wheel>
-    <!-- Rx sled: 15 kg, single centre wheel in front of a rear pair -->
+    <!-- Rx sled: 15 kg, single centre wheel in front of a rear pair; its wheels sit only 0.15 m below
+         its centre, so the body is 0.2 m tall to clear the ground -->
     <xacro:cart_body cart="rx_cart" parent="tx_cart_link" mass="15.0"
-                     length="1.0" width="0.6" height="0.3"
+                     length="1.0" width="0.6" height="0.2"
                      tow_x="-0.923" tow_z="-0.131" rod="3.3" front_x="0.58" front_z="0.066" />
     <xacro:cart_wheel cart="rx_cart" name="front">

Commit message: Remove the alignment run: mission laid out on the first fix, initial heading from line 1; cart model with pin joints and one effective axle per cart
Co-Authored-By: Claude Opus 5.5 (1M context) <noreply@anthropic.com>

File: scout_navigation/description/temrover_carts.xacro (robot description, xacro)
@@ -9,5 +9,5 @@
     <xacro:property name="yaw_limit" value="1.2" />
     <xacro:property name="pitch_limit" value="0.5" />
-    <xacro:macro name="cart_wheel" params="cart name *origin lateral_friction:=0.6">
+    <xacro:macro name="cart_wheel" params="cart name *origin">
         <link name="${cart}_${name}_wheel_link">
             <inertial>
@@ -35,8 +35,6 @@
         </joint>
         <gazebo reference="${cart}_${name}_wheel_link">
-            <!-- fdir1 in the wheel frame, so mu1 acts along the rolling direction -->
-            <fdir1>1 0 0</fdir1>
             <mu1>0.8</mu1>
-            <mu2>${lateral_friction}</mu2>
+            <mu2>0.8</mu2>
             <material>Gazebo/DarkGrey</material>
         </gazebo>
@@ -65,4 +63,19 @@
             <origin xyz="${tow_x} 0 ${tow_z}" />
         </joint>
+        <link name="${cart}_pivot_link">
+            <inertial>
+                <mass value="0.1" />
+                <inertia ixx="1e-4" ixy="0" ixz="0" iyy="1e-4" iyz="0" izz="1e-4" />
+            </inertial>
+        </link>
+        <joint name="${cart}_hitch_yaw" type="revolute">
+            <parent link="${cart}_tow_link" />
+            <child link="${cart}_pivot_link" />
+            <origin xyz="${-rod/2} 0 0" />
+            <axis xyz="0 0 1" />
+            <limit lower="${-yaw_limit}" upper="${yaw_limit}" effort="500" velocity="10" />
+            <dynamics damping="${yaw_damping}" />
+        </joint>
+        <!-- The pin also lets the cart's half pitch, so each cart stands on its own wheels -->
         <link name="${cart}_rod_link">
             <inertial>
@@ -79,11 +92,10 @@
             </visual>
         </link>
-        <joint name="${cart}_hitch_yaw" type="revolute">
-            <parent link="${cart}_tow_link" />
+        <joint name="${cart}_hitch_pitch" type="revolute">
+            <parent link="${cart}_pivot_link" />
             <child link="${cart}_rod_link" />
-            <origin xyz="${-rod/2} 0 0" />
-            <axis xyz="0 0 1" />
-            <limit lower="${-yaw_limit}" upper="${yaw_limit}" effort="500" velocity="10" />
-            <dynamics damping="${yaw_damping}" />
+            <axis xyz="0 1 0" />
+            <limit lower="${-pitch_limit}" upper="${pitch_limit}" effort="500" velocity="10" />
+            <dynamics damping="${pitch_damping}" />
         </joint>
         <link name="${cart}_link">
@@ -113,42 +125,32 @@
             </visual>
         </gazebo>
-        <joint name="${cart}_hitch_pitch" type="revolute">
+        <joint name="${cart}_frame" type="fixed">
             <parent link="${cart}_rod_link" />
             <child link="${cart}_link" />
             <origin xyz="${-rod/2-front_x} 0 ${front_z}" />
-            <axis xyz="0 1 0" />
-            <limit lower="${-pitch_limit}" upper="${pitch_limit}" effort="500" velocity="10" />
-            <dynamics damping="${pitch_damping}" />
         </joint>
     </xacro:macro>
-    <!-- Tx sled: 30 kg, four wheels, 0.8 m wheelbase -->
+    <!-- Each cart rolls on one effective axle at the middle of its real wheel set (Tx: four wheels on a
+         0.8 m wheelbase, Rx: one front wheel and a rear pair). With the pin that makes it a determinate
+         trailer, the same model turn_design.py uses; a rigid V on several fixed axles locks up in DART. -->
+    <!-- Tx sled: 30 kg -->
     <xacro:cart_body cart="tx_cart" parent="base_link" mass="30.0"
                      length="1.0" width="0.6" height="0.3"
                      tow_x="-0.47" tow_z="-0.05" rod="2.0" front_x="0.32" front_z="0.125" />
-    <xacro:cart_wheel cart="tx_cart" name="front_left">
-        <origin xyz="0.100 0.300 -0.215" />
+    <xacro:cart_wheel cart="tx_cart" name="left">
+        <origin xyz="-0.300 0.300 -0.215" />
     </xacro:cart_wheel>
-    <xacro:cart_wheel cart="tx_cart" name="front_right">
-        <origin xyz="0.100 -0.300 -0.215" />
+    <xacro:cart_wheel cart="tx_cart" name="right">
+        <origin xyz="-0.300 -0.300 -0.215" />
     </xacro:cart_wheel>
-    <xacro:cart_wheel cart="tx_cart" name="rear_left">
-        <origin xyz="-0.700 0.300 -0.215" />
-    </xacro:cart_wheel>
-    <xacro:cart_wheel cart="tx_cart" name="rear_right">
-        <origin xyz="-0.700 -0.300 -0.215" />
-    </xacro:cart_wheel>
-    <!-- Rx sled: 15 kg, single centre wheel in front of a rear pair; its wheels sit only 0.15 m below
-         its centre, so the body is 0.2 m tall to clear the ground -->
+    <!-- Rx sled: 15 kg; its wheels sit only 0.15 m below its centre, so the body is 0.2 m tall -->
     <xacro:cart_body cart="rx_cart" parent="tx_cart_link" mass="15.0"
                      length="1.0" width="0.6" height="0.2"
                      tow_x="-0.923" tow_z="-0.131" rod="3.3" front_x="0.58" front_z="0.066" />
-    <xacro:cart_wheel cart="rx_cart" name="front">
-        <origin xyz="0.330 0.0 -0.019" />
+    <xacro:cart_wheel cart="rx_cart" name="left">
+        <origin xyz="0.080 0.250 -0.019" />
     </xacro:cart_wheel>
-    <xacro:cart_wheel cart="rx_cart" name="rear_left">
-        <origin xyz="-0.170 0.250 -0.019" />
-    </xacro:cart_wheel>
-    <xacro:cart_wheel cart="rx_cart" name="rear_right">
-        <origin xyz="-0.170 -0.250 -0.019" />
+    <xacro:cart_wheel cart="rx_cart" name="right">
+        <origin xyz="0.080 -0.250 -0.019" />
     </xacro:cart_wheel>
 </robot>

Commit message: Plain U-turns with the towed carts, line-start wait, real line ends, Tx/Rx tracks and plots
- U-turn: a semicircle of half the line spacing (2.5 m), its far point 15 m past the line end;
  the run past each end now covers the Tx reaching the end and straightening
- Carts: front casters, fixed rear pair, link lengths from the build drawing, 90 deg hitch limit
- Navigator stops at each line's real start after a turn and waits for Start
  (wait_at_line_start), and latches survey_lines with the lines' real ends
- Gazebo marks the survey lines and their ends at launch from the site files; the static
  survey_path.sdf and make_path_marker.py are gone
- Dashboard: real line ends, dashed route, Rover/Tx/Rx tracks (replayed for a page opened
  mid-run), Tx-Rx separation and Rover-Tx offset plots against distance travelled
- turn_design.py settles on the Tx; research logs and architecture notes updated

Co-Authored-By: Claude Opus 5.5 (1M context) <noreply@anthropic.com>

File: scout_navigation/description/temrover_carts.xacro (robot description, xacro)
@@ -7,5 +7,6 @@
     <xacro:property name="yaw_damping" value="0.2" />
     <xacro:property name="pitch_damping" value="0.5" />
-    <xacro:property name="yaw_limit" value="1.2" />
+    <!-- Real PVC X-link limit not measured yet; 90 deg until it is -->
+    <xacro:property name="yaw_limit" value="${pi/2}" />
     <xacro:property name="pitch_limit" value="0.5" />
     <xacro:macro name="cart_wheel" params="cart name *origin">
@@ -40,6 +41,37 @@
         </gazebo>
     </xacro:macro>
+    <!-- Front casters swivel freely, so in the contact they only carry weight: frictionless spheres -->
+    <xacro:macro name="cart_caster" params="cart name *origin">
+        <link name="${cart}_${name}_caster_link">
+            <inertial>
+                <mass value="0.5" />
+                <inertia ixx="0.003" ixy="0" ixz="0" iyy="0.003" iyz="0" izz="0.003" />
+            </inertial>
+            <visual>
+                <geometry>
+                    <sphere radius="${cart_wheel_radius}" />
+                </geometry>
+            </visual>
+            <collision>
+                <geometry>
+                    <sphere radius="${cart_wheel_radius}" />
+                </geometry>
+            </collision>
+        </link>
+        <joint name="${cart}_${name}_caster" type="fixed">
+            <parent link="${cart}_link" />
+            <child link="${cart}_${name}_caster_link" />
+            <xacro:insert_block name="origin" />
+        </joint>
+        <gazebo reference="${cart}_${name}_caster_link">
+            <mu1>0.0</mu1>
+            <mu2>0.0</mu2>
+            <material>Gazebo/DarkGrey</material>
+        </gazebo>
+    </xacro:macro>
     <!-- Each PVC link is two rigid V frames pinned at its midpoint: the front half is fixed to the
-         towing unit, the yaw joint sits halfway, and the rear half pitches with the towed cart -->
+         towing unit, the yaw joint sits halfway, and the rear half pitches with the towed cart.
+         rover-Tx: an X of two 96 cm-sided Vs on a 25 cm base (0.952 m each half);
+         Tx-Rx: a 58 cm-sided V and a 107 cm rod each side of the pin (1.636 m each half) -->
     <xacro:macro name="cart_body" params="cart parent mass length width height
                                           tow_x tow_z rod front_x front_z">
@@ -131,26 +163,35 @@
         </joint>
     </xacro:macro>
-    <!-- Each cart rolls on one effective axle at the middle of its real wheel set (Tx: four wheels on a
-         0.8 m wheelbase, Rx: one front wheel and a rear pair). With the pin that makes it a determinate
-         trailer, the same model turn_design.py uses; a rigid V on several fixed axles locks up in DART. -->
+    <!-- Front wheels are casters and the rear pair is fixed, so each cart turns about its rear axle:
+         a determinate trailer, the same model turn_design.py uses. Tx: casters 0.8 m ahead of the
+         rear pair; Rx: one caster 0.5 m ahead of it. -->
     <!-- Tx sled: 30 kg -->
     <xacro:cart_body cart="tx_cart" parent="base_link" mass="30.0"
                      length="1.0" width="0.6" height="0.3"
-                     tow_x="-0.47" tow_z="-0.05" rod="2.0" front_x="0.32" front_z="0.125" />
+                     tow_x="-0.47" tow_z="-0.05" rod="1.904" front_x="0.32" front_z="0.125" />
     <xacro:cart_wheel cart="tx_cart" name="left">
-        <origin xyz="-0.300 0.300 -0.215" />
+        <origin xyz="-0.700 0.300 -0.215" />
     </xacro:cart_wheel>
     <xacro:cart_wheel cart="tx_cart" name="right">
-        <origin xyz="-0.300 -0.300 -0.215" />
+        <origin xyz="-0.700 -0.300 -0.215" />
     </xacro:cart_wheel>
+    <xacro:cart_caster cart="tx_cart" name="front_left">
+        <origin xyz="0.100 0.300 -0.215" />
+    </xacro:cart_caster>
+    <xacro:cart_caster cart="tx_cart" name="front_right">
+        <origin xyz="0.100 -0.300 -0.215" />
+    </xacro:cart_caster>
     <!-- Rx sled: 15 kg; its wheels sit only 0.15 m below its centre, so the body is 0.2 m tall -->
     <xacro:cart_body cart="rx_cart" parent="tx_cart_link" mass="15.0"
                      length="1.0" width="0.6" height="0.2"
-                     tow_x="-0.923" tow_z="-0.131" rod="3.3" front_x="0.58" front_z="0.066" />
+                     tow_x="-0.923" tow_z="-0.131" rod="3.272" front_x="0.58" front_z="0.066" />
     <xacro:cart_wheel cart="rx_cart" name="left">
-        <origin xyz="0.080 0.250 -0.019" />
+        <origin xyz="-0.170 0.250 -0.019" />
     </xacro:cart_wheel>
     <xacro:cart_wheel cart="rx_cart" name="right">
-        <origin xyz="0.080 -0.250 -0.019" />
+        <origin xyz="-0.170 -0.250 -0.019" />
     </xacro:cart_wheel>
+    <xacro:cart_caster cart="rx_cart" name="front">
+        <origin xyz="0.330 0 -0.019" />
+    </xacro:cart_caster>
 </robot>
